Commit message: Add RSI training and dumbbell grasp tooling

File: assets/urdf/ur5e_delto_description/ur5e_left_dg5f.urdf (robot description, URDF)
Before this commit: robot ur5e_left_dg5f, 39 links, 38 joints
Joints:
- joint lj_dg_1_3: limit lower=-1.5707963267948966 upper=0.0 effort=7.5 velocity=3.141592653589793 -> lower=-1.5707963267948966 upper=1.5707963267948966 effort=7.5 velocity=3.141592653589793
- joint lj_dg_5_2: limit lower=0.0 upper=0.4188790204786391 effort=7.5 velocity=3.141592653589793 -> lower=-0.6108652381980153 upper=0.4188790204786391 effort=7.5 velocity=3.141592653589793

File: assets/urdf/ur5e_delto_description/ur5e_right_dg5f.urdf (robot description, URDF)
Before this commit: robot ur5e_right_dg5f, 39 links, 38 joints
Joints:
- joint rj_dg_1_3: limit lower=-0.0 upper=1.5707963267948966 effort=7.5 velocity=3.141592653589793 -> lower=-1.5707963267948966 upper=1.5707963267948966 effort=7.5 velocity=3.141592653589793
- joint rj_dg_5_2: limit lower=-0.4188790204786391 upper=-0.0 effort=7.5 velocity=3.141592653589793 -> lower=-0.4188790204786391 upper=0.6108652381980153 effort=7.5 velocity=3.141592653589793
